Commit message: init

File: urdf/realsense-RS200.macro.xacro (robot description, xacro)
@@ -12,4 +12,5 @@
 <robot xmlns:xacro="http://ros.org/wiki/xacro">
 <xacro:macro name="realsense-rs200" params="prefix parent *origin">
+<xacro:arg name="prefix" default="camera_link"/>
     <!-- Camera link -->
     <link name="${prefix}rs200_camera">
@@ -17,5 +18,5 @@
             <origin rpy="0 0 0" xyz="0 0 0"/>
             <geometry>
-                <mesh filename="package://realsense_gazebo_plugin/models/realsense_camera/meshes/realsense.dae"/>
+                <mesh filename="package://rtabmap_drone_example/meshes/l515.dae"/>
             </geometry>
         </visual>
